Commit message: ros1-bridge working first commit

File: kmriiwa_description/urdf/iiwa14/iiwa14.xacro (robot description, xacro)
@@ -29,5 +29,5 @@
         <origin xyz="0 0 0" rpy="0 0 0"/>
         <geometry>
-          <mesh filename="package://kmriiwa_description/meshes/iiwa14/visual/link_0.stl"/>
+          <mesh filename="file://$(find kmriiwa_description)/meshes/iiwa14/visual/link_0.stl"/>
         </geometry>
         <material name="Grey"/>
@@ -36,5 +36,5 @@
         <origin xyz="0 0 0" rpy="0 0 0"/>
         <geometry>
-          <mesh filename="package://kmriiwa_description/meshes/iiwa14/collision/link_0.stl"/>
+          <mesh filename="file://$(find kmriiwa_description)/meshes/iiwa14/collision/link_0.stl"/>
         </geometry>
         <material name="Grey"/>
@@ -70,12 +70,12 @@
         <origin xyz="0 0 0" rpy="0 0 0"/>
         <geometry>
-          <mesh filename="package://kmriiwa_description/meshes/iiwa14/visual/link_1.stl"/>
-        </geometry>
-        <material name="Orange"/>
-      </visual>
-      <collision>
-        <origin xyz="0 0 0" rpy="0 0 0"/>
-        <geometry>
-          <mesh filename="package://kmriiwa_description/meshes/iiwa14/collision/link_1.stl"/>
+          <mesh filename="file://$(find kmriiwa_description)/meshes/iiwa14/visual/link_1.stl"/>
+        </geometry>
+        <material name="Orange"/>
+      </visual>
+      <collision>
+        <origin xyz="0 0 0" rpy="0 0 0"/>
+        <geometry>
+          <mesh filename="file://$(find kmriiwa_description)/meshes/iiwa14/collision/link_1.stl"/>
         </geometry>
         <material name="Orange"/>
@@ -105,12 +105,12 @@
         <origin xyz="0 0 0" rpy="0 0 0"/>
         <geometry>
-          <mesh filename="package://kmriiwa_description/meshes/iiwa14/visual/link_2.stl"/>
-        </geometry>
-        <material name="Orange"/>
-      </visual>
-      <collision>
-        <origin xyz="0 0 0" rpy="0 0 0"/>
-        <geometry>
-          <mesh filename="package://kmriiwa_description/meshes/iiwa14/collision/link_2.stl"/>
+          <mesh filename="file://$(find kmriiwa_description)/meshes/iiwa14/visual/link_2.stl"/>
+        </geometry>
+        <material name="Orange"/>
+      </visual>
+      <collision>
+        <origin xyz="0 0 0" rpy="0 0 0"/>
+        <geometry>
+          <mesh filename="file://$(find kmriiwa_description)/meshes/iiwa14/collision/link_2.stl"/>
         </geometry>
         <material name="Orange"/>
@@ -140,12 +140,12 @@
         <origin xyz="0 0 0" rpy="0 0 0"/>
         <geometry>
-          <mesh filename="package://kmriiwa_description/meshes/iiwa14/visual/link_3.stl"/>
-        </geometry>
-        <material name="Orange"/>
-      </visual>
-      <collision>
-        <origin xyz="0 0 0" rpy="0 0 0"/>
-        <geometry>
-          <mesh filename="package://kmriiwa_description/meshes/iiwa14/collision/link_3.stl"/>
+          <mesh filename="file://$(find kmriiwa_description)/meshes/iiwa14/visual/link_3.stl"/>
+        </geometry>
+        <material name="Orange"/>
+      </visual>
+      <collision>
+        <origin xyz="0 0 0" rpy="0 0 0"/>
+        <geometry>
+          <mesh filename="file://$(find kmriiwa_description)/meshes/iiwa14/collision/link_3.stl"/>
         </geometry>
         <material name="Orange"/>
@@ -175,12 +175,12 @@
         <origin xyz="0 0 0" rpy="0 0 0"/>
         <geometry>
-          <mesh filename="package://kmriiwa_description/meshes/iiwa14/visual/link_4.stl"/>
-        </geometry>
-        <material name="Orange"/>
-      </visual>
-      <collision>
-        <origin xyz="0 0 0" rpy="0 0 0"/>
-        <geometry>
-          <mesh filename="package://kmriiwa_description/meshes/iiwa14/collision/link_4.stl"/>
+          <mesh filename="file://$(find kmriiwa_description)/meshes/iiwa14/visual/link_4.stl"/>
+        </geometry>
+        <material name="Orange"/>
+      </visual>
+      <collision>
+        <origin xyz="0 0 0" rpy="0 0 0"/>
+        <geometry>
+          <mesh filename="file://$(find kmriiwa_description)/meshes/iiwa14/collision/link_4.stl"/>
         </geometry>
         <material name="Orange"/>
@@ -210,12 +210,12 @@
         <origin xyz="0 0 0" rpy="0 0 0"/>
         <geometry>
-          <mesh filename="package://kmriiwa_description/meshes/iiwa14/visual/link_5.stl"/>
-        </geometry>
-        <material name="Orange"/>
-      </visual>
-      <collision>
-        <origin xyz="0 0 0" rpy="0 0 0"/>
-        <geometry>
-          <mesh filename="package://kmriiwa_description/meshes/iiwa14/collision/link_5.stl"/>
+          <mesh filename="file://$(find kmriiwa_description)/meshes/iiwa14/visual/link_5.stl"/>
+        </geometry>
+        <material name="Orange"/>
+      </visual>
+      <collision>
+        <origin xyz="0 0 0" rpy="0 0 0"/>
+        <geometry>
+          <mesh filename="file://$(find kmriiwa_description)/meshes/iiwa14/collision/link_5.stl"/>
         </geometry>
         <material name="Orange"/>
@@ -245,12 +245,12 @@
         <origin xyz="0 0 0" rpy="0 0 0"/>
         <geometry>
-          <mesh filename="package://kmriiwa_description/meshes/iiwa14/visual/link_6.stl"/>
-        </geometry>
-        <material name="Orange"/>
-      </visual>
-      <collision>
-        <origin xyz="0 0 0" rpy="0 0 0"/>
-        <geometry>
-          <mesh filename="package://kmriiwa_description/meshes/iiwa14/collision/link_6.stl"/>
+          <mesh filename="file://$(find kmriiwa_description)/meshes/iiwa14/visual/link_6.stl"/>
+        </geometry>
+        <material name="Orange"/>
+      </visual>
+      <collision>
+        <origin xyz="0 0 0" rpy="0 0 0"/>
+        <geometry>
+          <mesh filename="file://$(find kmriiwa_description)/meshes/iiwa14/collision/link_6.stl"/>
         </geometry>
         <material name="Orange"/>
@@ -280,5 +280,5 @@
         <origin xyz="0 0 0" rpy="0 0 0"/>
         <geometry>
-          <mesh filename="package://kmriiwa_description/meshes/iiwa14/visual/link_7.stl"/>
+          <mesh filename="file://$(find kmriiwa_description)/meshes/iiwa14/visual/link_7.stl"/>
         </geometry>
         <material name="Grey"/>
@@ -287,5 +287,5 @@
         <origin xyz="0 0 0" rpy="0 0 0"/>
         <geometry>
-          <mesh filename="package://kmriiwa_description/meshes/iiwa14/collision/link_7.stl"/>
+          <mesh filename="file://$(find kmriiwa_description)/meshes/iiwa14/collision/link_7.stl"/>
         </geometry>
         <material name="Grey"/>

File: kmriiwa_description/urdf/kmp200/kmp200.xacro (robot description, xacro)
@@ -1,4 +1,5 @@
 <?xml version="1.0"?>
 <robot xmlns:xacro="http://www.ros.org/wiki/xacro">
+<!-- TODO Make relative import for the mesh file, I am tired of not getting meshes, or put all the description in the main src file and use $(find package_name) -->
   <!-- Import Gazebo-settings -->
   <xacro:include filename="$(find kmriiwa_description)/urdf/kmp200/kmp200.gazebo.xacro" />
@@ -25,5 +26,5 @@
         <visual>
           <geometry>
-            <mesh filename="package://kmriiwa_description/meshes/kmp200/KMP200.dae"/>
+            <mesh filename="file://$(find kmriiwa_description)/meshes/kmp200/KMP200.dae"/>
           </geometry>
           <material name="White"/>
@@ -31,5 +32,5 @@
         <collision>
           <geometry>
-            <mesh filename="package://kmriiwa_description/meshes/kmp200/KMP200.dae"/>
+            <mesh filename="file://$(find kmriiwa_description)/meshes/kmp200/KMP200.dae"/>
           </geometry>
         </collision>
@@ -56,5 +57,5 @@
           <origin xyz="0 0 0" rpy="3.1413 0 0"/>
           <geometry>
-              <mesh filename="package://kmriiwa_description/meshes/kmp200/sensors/visual/sick_lms1xx.dae" />
+              <mesh filename="file://$(find kmriiwa_description)/meshes/kmp200/sensors/visual/sick_lms1xx.dae" />
           </geometry>
           <material name="DarkGrey"/>
@@ -63,5 +64,5 @@
             <origin xyz="0.0 0 0.0" rpy="0 0 0"/>
             <geometry>
-                <mesh filename="package://kmriiwa_description/meshes/kmp200/sensors/collision/sick_lms1xx.stl" />
+                <mesh filename="file://$(find kmriiwa_description)/meshes/kmp200/sensors/collision/sick_lms1xx.stl" />
             </geometry>
         </collision>
@@ -80,5 +81,5 @@
           <origin xyz="0.0 0 0" rpy="0 3.1413 3.1413"/>
           <geometry>
-              <mesh filename="package://kmriiwa_description/meshes/kmp200/sensors/visual/sick_lms1xx.dae" />
+              <mesh filename="file://$(find kmriiwa_description)/meshes/kmp200/sensors/visual/sick_lms1xx.dae" />
           </geometry>
           <material name="DarkGrey"/>
@@ -87,5 +88,5 @@
             <origin xyz="0 0 0" rpy="0 0 0"/>
             <geometry>
-                  <mesh filename="package://kmriiwa_description/meshes/kmp200/sensors/collision/sick_lms1xx.stl" />
+                  <mesh filename="file://$(find kmriiwa_description)/meshes/kmp200/sensors/collision/sick_lms1xx.stl" />
             </geometry>
         </collision>
@@ -99,5 +100,5 @@
           <origin xyz="0 0 0" rpy="0 0 0" />
           <geometry>
-            <mesh filename="package://kmriiwa_description/meshes/kmp200/wheels/omni_wheel_1.dae" scale="1.06695 1.06695 1.06695"/>
+            <mesh filename="file://$(find kmriiwa_description)/meshes/kmp200/wheels/omni_wheel_1.dae" scale="1.06695 1.06695 1.06695"/>
           </geometry>
         </visual>
@@ -113,5 +114,5 @@
           <origin xyz="0 0 0" rpy="0 0 0" />
           <geometry>
-            <mesh filename="package://kmriiwa_description/meshes/kmp200/wheels/omni_wheel_1.dae" scale="1.06695 1.06695 1.06695"/>
+            <mesh filename="file://$(find kmriiwa_description)/meshes/kmp200/wheels/omni_wheel_1.dae" scale="1.06695 1.06695 1.06695"/>
           </geometry>
         </visual>
@@ -127,5 +128,5 @@
           <origin xyz="0 0 0" rpy="0 0 0" />
           <geometry>
-            <mesh filename="package://kmriiwa_description/meshes/kmp200/wheels/omni_wheel_1.dae" scale="1.06695 1.06695 1.06695"/>
+            <mesh filename="file://$(find kmriiwa_description)/meshes/kmp200/wheels/omni_wheel_1.dae" scale="1.06695 1.06695 1.06695"/>
           </geometry>
         </visual>
@@ -141,5 +142,5 @@
           <origin xyz="0 0 0" rpy="0 0 0" />
           <geometry>
-            <mesh filename="package://kmriiwa_description/meshes/kmp200/wheels/omni_wheel_1.dae" scale="1.06695 1.06695 1.06695"/>
+            <mesh filename="file://$(find kmriiwa_description)/meshes/kmp200/wheels/omni_wheel_1.dae" scale="1.06695 1.06695 1.06695"/>
           </geometry>
         </visual>

File: kmriiwa_description/urdf/robot/kmriiwa.urdf.xacro (robot description, xacro)
@@ -11,6 +11,6 @@
   <xacro:property name="arm_base_flange_z_pos" value="-0.01" />
   <xacro:property name="arm_base_flange_yew" value="-1.5708" />
-  <xacro:property name="riser_flange_height" value="0.26" />
-  <xacro:property name="riser_flange_radius" value="0.121" />
+  <xacro:property name="riser_flange_height" value="0.0" />   <!--Changed stuff here and made zero -->
+  <xacro:property name="riser_flange_radius" value="0.0" />
   <xacro:property name="flange_origin_xyz" value="${arm_base_flange_x_pos} ${arm_base_flange_y_pos} ${arm_base_flange_z_pos+riser_flange_height/2}"/>
   <xacro:property name="flange_origin_rpy" value="0 0 ${arm_base_flange_yew}"/>
