Commit message: Minor changes to seventh axis movement

File: kmriiwa_description/urdf/robot/working_kdl_urdf/kmriiwakdl.urdf (robot description, URDF)
Before this commit: robot kmriiwa, 23 links, 22 joints
Links:
- removed link camera_color_optical_frame_tf
- removed link kmriiwa_camera_link
- removed link kmriiwa_gripper_link
- removed link kmriiwa_gripper_tcp
Joints:
- removed joint kmriiwa_camera_joint
- removed joint kmriiwa_gripper_joint
- removed joint kmriiwa_gripper_tcp_joint
- removed joint kmriiwa_realsense_frame_joint

File: kmriiwa_description/urdf/robot_extras/robot_extras.xacro (robot description, xacro)
@@ -53,10 +53,10 @@
     </link>
     <!-- Frame for realsense camera here- only frame here -->
-    <joint name="${robot_name}_gripper_tcp_joint" type="fixed">
-      <parent link="${robot_name}_gripper_link"/>
-      <child link="${robot_name}_gripper_tcp"/>
-      <origin xyz="0 0 0.2" rpy="${-90.0 * pi/180}  0  ${120.0 * pi/180}"/> <!-- Adjust position as needed -->
+    <joint name="${robot_name}_realsense_frame_joint" type="fixed">
+      <parent link="${robot_name}_camera_link"/>
+      <child link="camera_color_optical_frame_tf"/>
+      <origin xyz="0 0.07 0.0" rpy="0 ${-90.0 * pi/180} 0"/> <!-- Adjust position as needed -->
     </joint>
-    <link name="${robot_name}_gripper_tcp"/>
+    <link name="camera_color_optical_frame_tf"/>
   </xacro:macro>
 </robot>
